File: Hardware/H616_DDR3/_restore_backup_2026-08-15T11-41-33-522/dram.kicad_sch (KiCad schematic)
At the start: 26 parts, among them U1 H616, U2 K4B8G1646D

Commit message: v
Parts:
- R5: now not fitted
Changed lines of the file:
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@@
 		(on_board yes)
 		(in_pos_files yes)
-		(dnp no)
+		(dnp yes)
 		(fields_autoplaced yes)
 		(property "Reference" "R5"
