File: Hardware/H616_DDR3/_restore_backup_2026-08-15T11-41-33-522/io1.kicad_sch (KiCad schematic)
At the start: 16 parts, among them U1 H616, Y1 24MHz

Commit message: v
Parts:
- removed C54, C55: 470n, Capacitor_SMD:C_0402_1005Metric_Pad0.74x0.62mm_HandSolder, symbol Device:C
- removed C56: 2.2u, Capacitor_SMD:C_0402_1005Metric_Pad0.74x0.62mm_HandSolder, symbol Device:C
- removed C57: 1u, Capacitor_SMD:C_0402_1005Metric_Pad0.74x0.62mm_HandSolder, symbol Device:C
- removed C58, C61, C62, C70: 100n, Capacitor_SMD:C_0402_1005Metric_Pad0.74x0.62mm_HandSolder, symbol Device:C
- removed C59, C60: 18p, Capacitor_SMD:C_0402_1005Metric_Pad0.74x0.62mm_HandSolder, symbol Device:C
- removed C63: 220n, Capacitor_SMD:C_0402_1005Metric_Pad0.74x0.62mm_HandSolder, symbol Device:C
- removed C64: 1n, Capacitor_SMD:C_0402_1005Metric_Pad0.74x0.62mm_HandSolder, symbol Device:C
- removed R19: 150k, Resistor_SMD:R_0402_1005Metric_Pad0.72x0.64mm_HandSolder, symbol Device:R
- removed R20: 10k, Resistor_SMD:R_0402_1005Metric_Pad0.72x0.64mm_HandSolder, symbol Device:R
- removed U1: H616, projectlib:H616_TFBGA284, symbol H616_lib:H616
- removed Y1: 24MHz, Crystal:Crystal_SMD_2520-4Pin_2.5x2.0mm, symbol Device:Crystal_GND24_Small
- added C51: 10u, Capacitor_SMD:C_0402_1005Metric_Pad0.74x0.62mm_HandSolder, symbol Device:C
- added C52, C53: 2.2u, Capacitor_SMD:C_0402_1005Metric_Pad0.74x0.62mm_HandSolder, symbol Device:C
- added D1, D2: LED, LED_SMD:LED_0603_1608Metric_Pad1.05x0.95mm_HandSolder, symbol Device:LED
- added J1: Micro_SD_Card_Det2, Connector_Card:microSD_HC_Hirose_DM3AT-SF-PEJM5, symbol Connector:Micro_SD_Card_Det2
- added R10: 1R, Resistor_SMD:R_0402_1005Metric_Pad0.72x0.64mm_HandSolder, symbol Device:R
- added R11: 33R, Resistor_SMD:R_0402_1005Metric_Pad0.72x0.64mm_HandSolder, symbol Device:R
- added R12, R13, R26: 10k, Resistor_SMD:R_0402_1005Metric_Pad0.72x0.64mm_HandSolder, symbol Device:R
- added R14: 1k, Resistor_SMD:R_0402_1005Metric_Pad0.72x0.64mm_HandSolder, symbol Device:R
- added R15, R16, R17, R18: 2k, Resistor_SMD:R_0402_1005Metric_Pad0.72x0.64mm_HandSolder, symbol Device:R
- added TP11, TP12, TP13: TestPoint, TestPoint:TestPoint_THTPad_D1.0mm_Drill0.5mm, symbol Connector:TestPoint
- added U1: H616, projectlib:H616_TFBGA284, symbol H616_lib:H616
Connections:
- net +1V8: now also C53.1, R17.2, R18.2, U1.D7 (VCC_PG)
- net +3.3V: now also C51.1, C52.1, R10.2, R12.2, R13.2, R26.2, U1.F5 (VCC_PC), U1.J6 (VCC_PI)
- net GND: now also C51.2, C52.2, C53.2, D1.1 (K), D2.1 (K), J1.10 (DET_A), J1.11 (SHIELD), J1.6 (VSS), R14.1
- new net: J1.5 (CLK), R11.1
- new net: R26.1, U1.D1 (PC3)
- new net: TP11.1, U1.D2 (PC4)
- new net: TP12.1, U1.D3 (PC5)
- new net: TP13.1, U1.E2 (PC6)
- new net: R15.2, U1.G2 (PC12)
- new net: R16.2, U1.G3 (PC13)
- new net: D1.2 (A), R15.1
- new net: D2.2 (A), R16.1
- new net CLK125: U1.E5 (PI13)
- new net MDC: U1.L6 (PI14)
- new net MDIO: U1.L4 (PI15)
- new net PMU_SCK: R17.1, U1.C18 (PL0)
- new net PMU_SDA: R18.1, U1.B18 (PL1)
- new net RXC: U1.G5 (PI4)
- new net RXCTL: U1.H4 (PI5)
- new net RXConvIn: U1.D16 (PH0)
- new net RXD0: U1.E4 (PI3)
- new net RXD1: U1.G6 (PI2)
- new net RXD2: U1.D4 (PI1)
- new net RXD3: U1.H6 (PI0)
- new net SDC0_CLK: R11.2, U1.K1 (PF2)
- new net SDC0_CMD: J1.3 (CMD), R12.1, U1.K3 (PF3)
- new net SDC0_D0: J1.7 (DAT0), U1.J3 (PF1)
- new net SDC0_D1: J1.8 (DAT1), U1.J2 (PF0)
- new net SDC0_D2: J1.1 (DAT2), U1.L3 (PF5)
- new net SDC0_D3: J1.2 (DAT3/CD), U1.L2 (PF4)
- new net SDC0_DET: J1.9 (DET_B), R13.1, R14.2, U1.K2 (PF6)
- new net SD_VDD: J1.4 (VDD), R10.1
- new net TXC: U1.K4 (PI11)
- new net TXCTL: U1.K5 (PI12)
- new net TXConvOut: U1.D15 (PH1)
- new net TXD0: U1.L5 (PI10)
- new net TXD1: U1.D5 (PI9)
- new net TXD2: U1.E6 (PI8)
- new net TXD3: U1.G4 (PI7)
- no-connect marks 25 -> 39
