File: Hardware/H616_DDR3/_restore_backup_2026-08-15T11-41-33-522/power.kicad_sch (KiCad schematic)
At the start: 55 parts, among them U1 H616, U3 AXP305

Commit message: v
Parts:
- added TP10, TP9: TestPoint, TestPoint:TestPoint_THTPad_D1.0mm_Drill0.5mm, symbol Connector:TestPoint
Connections:
- net GND: now also TP10.1, TP9.1
