File: Hardware/H616_DDR3/charge.kicad_sch (KiCad schematic)
At the start: 22 parts, among them J4 USB_C_Receptacle_USB2.0, Q1 AO3420_C358680, SW1 CK_KMS2xxG, U4 SW6206, U5 BX-PH2_0-2PZZ

Commit message: trace
Parts:
- U4: footprint Package_DFN_QFN:QFN-48-1EP_6x6mm_P0.4mm_EP4.2x4.2mm -> Package_DFN_QFN:QFN-48-1EP_6x6mm_P0.4mm_EP4.2x4.2mm_ThermalVias
Changed lines of the file:
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@@
 			)
 		)
-		(property "Footprint" "Package_DFN_QFN:QFN-48-1EP_6x6mm_P0.4mm_EP4.2x4.2mm"
+		(property "Footprint" "Package_DFN_QFN:QFN-48-1EP_6x6mm_P0.4mm_EP4.2x4.2mm_ThermalVias"
 			(at 120.65 80.01 0)
 			(hide yes)

Commit message: trace
Parts:
- removed BT1: Battery_Cell, symbol Device:Battery_Cell
- U5: now not fitted
Changed lines of the file:
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@@
-	)
-	(junction
-		(at 31.75 52.07)
-		(diameter 0)
-		(color 0 0 0 0)
 	)
 	(junction
@@
 	(wire
 		(pts
-			(xy 29.21 52.07) (xy 31.75 52.07)
+			(xy 29.21 52.07) (xy 48.26 52.07)
 		)
 		(stroke
@@
 		(pts
 			(xy 154.94 96.52) (xy 182.88 96.52)
-		)
-		(stroke
-			(width 0)
-			(type default)
-		)
-	)
-	(wire
-		(pts
-			(xy 31.75 52.07) (xy 48.26 52.07)
 		)
 		(stroke
@@
 		(exclude_from_sim no)
 		(in_bom yes)
-		(on_board yes)
+		(on_board no)
 		(in_pos_files yes)
-		(dnp no)
+		(dnp yes)
 		(fields_autoplaced yes)
 		(property "Reference" "U5"
@@
 					(unit 1)
 				)
-			)
-		)
-	)
-	(symbol
-		(lib_id "Device:Battery_Cell")
-		(at 31.75 57.15 0)
-		(unit 1)
-		(body_style 1)
-		(exclude_from_sim no)
-		(in_bom yes)
-		(on_board yes)
-		(in_pos_files yes)
-		(dnp no)
-		(fields_autoplaced yes)
-		(property "Reference" "BT1"
-			(at 35.56 54.0384 0)
-			(show_name no)
-			(do_not_autoplace no)
-			(effects
-				(font
-					(size 1.27 1.27)
-				)
-				(justify left)
-			)
-		)
-		(property "Value" "Battery_Cell"
-			(at 35.56 56.5784 0)
-			(show_name no)
-			(do_not_autoplace no)
-			(effects
-				(font
-					(size 1.27 1.27)
-				)
-				(justify left)
-			)
-		)
-		(property "Footprint" ""
-			(at 31.75 55.626 90)
-			(hide yes)
-			(show_name no)
-			(do_not_autoplace no)
-			(effects
-				(font
-					(size 1.27 1.27)
-				)
-			)
-		)
-		(property "Datasheet" ""
-			(at 31.75 55.626 90)
-			(hide yes)
-			(show_name no)
-			(do_not_autoplace no)
-			(effects
-				(font
-					(size 1.27 1.27)
-				)
-			)
-		)
-		(property "Description" "Single-cell battery"
-			(at 31.75 57.15 0)
-			(hide yes)
-			(show_name no)
-			(do_not_autoplace no)
-			(effects
-				(font
-					(size 1.27 1.27)
-				)
-			)
-		)
-		(property "Sim.Device" "V"
-			(at 31.75 57.15 0)
-			(hide yes)
-			(show_name no)
-			(do_not_autoplace no)
-			(effects
-				(font
-					(size 1.27 1.27)
-				)
-			)
-		)
-		(property "Sim.Type" "DC"
-			(at 31.75 57.15 0)
-			(hide yes)
-			(show_name no)
-			(do_not_autoplace no)
-			(effects
-				(font
-					(size 1.27 1.27)
-				)
-			)
-		)
-		(property "Sim.Pins" "1=+ 2=-"
-			(at 31.75 57.15 0)
-			(hide yes)
-			(show_name no)
-			(do_not_autoplace no)
-			(effects
-				(font
-					(size 1.27 1.27)
-				)
-			)
-		)
-		(pin "2"
-		)
-		(pin "1"
-		)
-		(instances
-			(project "H616_devboard"
-				(path "/44f68964-8d75-4db0-b784-705712e148bc/34c0604f-0eea-4ed0-a3f4-7af63e92cae5"
-					(reference "BT1")
-					(unit 1)
-				)

Commit message: buttons, pcb
Parts:
- SW1: footprint Button_Switch_SMD:SW_SPST_CK_KMS2xxGP -> bodya:button 3x6x3.5mm
Connections:
- net at R28.1, U4.20 (KEY/GSET): now also SW1.4; no longer SW1.2
Changed lines of the file:
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@@
 	)
 	(junction
-		(at 88.9 97.79)
-		(diameter 0)
-		(color 0 0 0 0)
-	)
-	(junction
 		(at 101.6 59.69)
 		(diameter 0)
@@
 	)
 	(junction
+		(at 88.9 97.79)
+		(diameter 0)
+		(color 0 0 0 0)
+	)
+	(junction
 		(at 101.6 52.07)
 		(diameter 0)
@@
 	(wire
 		(pts
-			(xy 71.12 97.79) (xy 76.2 97.79)
+			(xy 64.77 97.79) (xy 68.58 97.79)
 		)
 		(stroke
@@
 	(wire
 		(pts
-			(xy 86.36 97.79) (xy 88.9 97.79)
+			(xy 78.74 97.79) (xy 88.9 97.79)
 		)
 		(stroke
@@
 	(symbol
 		(lib_id "power:GND")
-		(at 71.12 97.79 270)
+		(at 64.77 97.79 270)
 		(unit 1)
 		(body_style 1)
@@
 		(fields_autoplaced yes)
 		(property "Reference" "#PWR0105"
-			(at 64.77 97.79 0)
+			(at 58.42 97.79 0)
 			(hide yes)
 			(show_name no)
@@
 		)
 		(property "Value" "GND"
-			(at 67.31 97.7899 90)
+			(at 60.96 97.7899 90)
 			(show_name no)
 			(do_not_autoplace no)
@@
 		)
 		(property "Footprint" ""
-			(at 71.12 97.79 0)
+			(at 64.77 97.79 0)
 			(hide yes)
 			(show_name no)
@@
 		)
 		(property "Datasheet" ""
-			(at 71.12 97.79 0)
+			(at 64.77 97.79 0)
 			(hide yes)
 			(show_name no)
@@
 		)
 		(property "Description" "Power symbol creates a global label with name \"GND\" , ground"
-			(at 71.12 97.79 0)
+			(at 64.77 97.79 0)
 			(hide yes)
 			(show_name no)
@@
 	(symbol
 		(lib_id "Switch:CK_KMS2xxG")
-		(at 81.28 97.79 0)
+		(at 73.66 97.79 0)
 		(unit 1)
 		(body_style 1)
@@
 		(fields_autoplaced yes)
 		(property "Reference" "SW1"
-			(at 81.28 90.17 0)
+			(at 73.66 90.17 0)
 			(show_name no)
 			(do_not_autoplace no)
@@
 		)
 		(property "Value" "CK_KMS2xxG"
-			(at 81.28 92.71 0)
+			(at 73.66 92.71 0)
 			(show_name no)
 			(do_not_autoplace no)
@@
 			)
 		)
-		(property "Footprint" "Button_Switch_SMD:SW_SPST_CK_KMS2xxGP"
-			(at 81.28 92.71 0)
+		(property "Footprint" "bodya:button 3x6x3.5mm"
+			(at 73.66 92.71 0)
 			(hide yes)
 			(show_name no)
@@
 		)
 		(property "Datasheet" "https://www.ckswitches.com/media/1482/kms.pdf"
-			(at 81.28 92.71 0)
+			(at 73.66 92.71 0)
 			(hide yes)
 			(show_name no)
@@
 		)
 		(property "Description" "Microminiature SMT Side Actuated, 4.2 x 2.8 x 1.42mm, without pegs, with shield pin"
-			(at 81.28 97.79 0)
+			(at 73.66 97.79 0)
 			(hide yes)
 			(show_name no)
@@
 		(pin "1"
 		)
-		(pin "2"
+		(pin "4"
+		)
+		(pin "SH"
 		)
 		(pin "SH"

Commit message: Errors fix
Connections:
- net GND: now also SW1.SH (3)
Other:
- moved on the sheet: SW1
Changed lines of the file:
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@@
 	(wire
 		(pts
+			(xy 67.31 93.98) (xy 67.31 97.79)
+		)
+		(stroke
+			(width 0)
+			(type default)
+		)
+	)
+	(wire
+		(pts
 			(xy 248.92 139.7) (xy 251.46 139.7)
 		)
@@
 	(wire
 		(pts
-			(xy 64.77 97.79) (xy 68.58 97.79)
+			(xy 67.31 93.98) (xy 68.58 93.98)
 		)
 		(stroke
@@
 	(wire
 		(pts
+			(xy 88.9 93.98) (xy 88.9 97.79)
+		)
+		(stroke
+			(width 0)
+			(type default)
+		)
+	)
+	(wire
+		(pts
 			(xy 248.92 137.16) (xy 251.46 137.16)
 		)
@@
 	(wire
 		(pts
-			(xy 78.74 97.79) (xy 88.9 97.79)
+			(xy 78.74 93.98) (xy 88.9 93.98)
 		)
 		(stroke
@@
 	(wire
 		(pts
+			(xy 67.31 97.79) (xy 64.77 97.79)
+		)
+		(stroke
+			(width 0)
+			(type default)
+		)
+	)
+	(wire
+		(pts
 			(xy 88.9 97.79) (xy 101.6 97.79)
 		)
@@
 	)
 	(symbol
+		(lib_id "power:GND")
+		(at 73.66 97.79 0)
+		(unit 1)
+		(body_style 1)
+		(exclude_from_sim no)
+		(in_bom yes)
+		(on_board yes)
+		(in_pos_files yes)
+		(dnp no)
+		(fields_autoplaced yes)
+		(property "Reference" "#PWR016"
+			(at 73.66 104.14 0)
+			(hide yes)
+			(show_name no)
+			(do_not_autoplace no)
+			(effects
+				(font
+					(size 1.27 1.27)
+				)
+			)
+		)
+		(property "Value" "GND"
+			(at 73.66 102.87 0)
+			(show_name no)
+			(do_not_autoplace no)
+			(effects
+				(font
+					(size 1.27 1.27)
+				)
+			)
+		)
+		(property "Footprint" ""
+			(at 73.66 97.79 0)
+			(hide yes)
+			(show_name no)
+			(do_not_autoplace no)
+			(effects
+				(font
+					(size 1.27 1.27)
+				)
+			)
+		)
+		(property "Datasheet" ""
+			(at 73.66 97.79 0)
+			(hide yes)
+			(show_name no)
+			(do_not_autoplace no)
+			(effects
+				(font
+					(size 1.27 1.27)
+				)
+			)
+		)
+		(property "Description" "Power symbol creates a global label with name \"GND\" , ground"
+			(at 73.66 97.79 0)
+			(hide yes)
+			(show_name no)
+			(do_not_autoplace no)
+			(effects
+				(font
+					(size 1.27 1.27)
+				)
+			)
+		)
+		(pin "1"
+		)
+		(instances
+			(project "H616_devboard"
+				(path "/44f68964-8d75-4db0-b784-705712e148bc/34c0604f-0eea-4ed0-a3f4-7af63e92cae5"
+					(reference "#PWR016")
+					(unit 1)
+				)
+			)
+		)
+	)
+	(symbol
 		(lib_id "Device:C")
 		(at 154.94 77.47 90)
@@
 	(symbol
 		(lib_id "power:GND")
+		(at 76.2 97.79 0)
+		(unit 1)
+		(body_style 1)
+		(exclude_from_sim no)
+		(in_bom yes)
+		(on_board yes)
+		(in_pos_files yes)
+		(dnp no)
+		(fields_autoplaced yes)
+		(property "Reference" "#PWR042"
+			(at 76.2 104.14 0)
+			(hide yes)
+			(show_name no)
+			(do_not_autoplace no)
+			(effects
+				(font
+					(size 1.27 1.27)
+				)
+			)
+		)
+		(property "Value" "GND"
+			(at 76.2 102.87 0)
+			(show_name no)
+			(do_not_autoplace no)
+			(effects
+				(font
+					(size 1.27 1.27)
+				)
+			)
+		)
+		(property "Footprint" ""
+			(at 76.2 97.79 0)
+			(hide yes)
+			(show_name no)
+			(do_not_autoplace no)
+			(effects
+				(font
+					(size 1.27 1.27)
+				)
+			)
+		)
+		(property "Datasheet" ""
+			(at 76.2 97.79 0)
+			(hide yes)
+			(show_name no)
+			(do_not_autoplace no)
+			(effects
+				(font
+					(size 1.27 1.27)
+				)
+			)
+		)
+		(property "Description" "Power symbol creates a global label with name \"GND\" , ground"
+			(at 76.2 97.79 0)
+			(hide yes)
+			(show_name no)
+			(do_not_autoplace no)
+			(effects
+				(font
+					(size 1.27 1.27)
+				)
+			)
+		)
+		(pin "1"
+		)
+		(instances
+			(project "H616_devboard"
+				(path "/44f68964-8d75-4db0-b784-705712e148bc/34c0604f-0eea-4ed0-a3f4-7af63e92cae5"
+					(reference "#PWR042")
+					(unit 1)
+				)
+			)
+		)
+	)
+	(symbol
+		(lib_id "power:GND")
 		(at 63.5 63.5 0)
 		(unit 1)
@@
 	(symbol
 		(lib_id "Switch:CK_KMS2xxG")
-		(at 73.66 97.79 0)
+		(at 73.66 93.98 0)
 		(unit 1)
 		(body_style 1)
@@
 		(fields_autoplaced yes)
 		(property "Reference" "SW1"
-			(at 73.66 90.17 0)
+			(at 73.66 86.36 0)
 			(show_name no)
 			(do_not_autoplace no)
@@
 		)
 		(property "Value" "CK_KMS2xxG"
-			(at 73.66 92.71 0)
+			(at 73.66 88.9 0)
 			(show_name no)
 			(do_not_autoplace no)
@@
 		)
 		(property "Footprint" "bodya:button 3x6x3.5mm"
-			(at 73.66 92.71 0)
+			(at 73.66 88.9 0)
 			(hide yes)
 			(show_name no)
@@
 		)
 		(property "Datasheet" "https://www.ckswitches.com/media/1482/kms.pdf"
-			(at 73.66 92.71 0)
+			(at 73.66 88.9 0)
 			(hide yes)
 			(show_name no)
@@
 		)
 		(property "Description" "Microminiature SMT Side Actuated, 4.2 x 2.8 x 1.42mm, without pegs, with shield pin"
-			(at 73.66 97.79 0)
+			(at 73.66 93.98 0)
 			(hide yes)
 			(show_name no)
