File: Hardware/H616_DDR3/dram.kicad_sch (KiCad schematic)
At the start: 26 parts, among them U1 H616, U2 K4B8G1646D

Commit message: radio+hdr
Parts:
- added C86, C87, C88: 1u, Capacitor_SMD:C_0402_1005Metric, symbol Device:C
- C1, C10, C11, C12, C13, C14, C2, C3, C4, C5, C6, C66, C67, C68, C69, C7, C8, C9: footprint Capacitor_SMD:C_0402_1005Metric_Pad0.74x0.62mm_HandSolder -> Capacitor_SMD:C_0402_1005Metric
- R1, R2, R3, R4, R5, R6: footprint Resistor_SMD:R_0402_1005Metric_Pad0.72x0.64mm_HandSolder -> Resistor_SMD:R_0402_1005Metric
Connections:
- net GND: now also C66.2, C67.2, C68.2, C69.2, C86.2, C87.2, C88.2
- net VCC_DRAM: now also C86.1, C87.1, C88.1
Other:
- moved on the sheet: C67, C69
