File: Hardware/H616_DDR3/H616_devboard.kicad_sch (KiCad schematic)
At the start: 0 parts

Commit message: Fix critical hardware bugs: eMMC HS400, AXP305 power rails, SW6206 Kelvin sense, Type-C CC and hierarchy
Other:
- added sheet BOARD (board.kicad_sch)
- added sheet CHARGE (charge.kicad_sch)
Changed lines of the file:
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@@
+		)
+	)
+	(sheet
+		(at 174.625 109.22)
+		(size 27.94 22.86)
+		(exclude_from_sim no)
+		(in_bom yes)
+		(on_board yes)
+		(dnp no)
+		(fields_autoplaced yes)
+		(stroke
+			(width 0.1524)
+			(type solid)
+		)
+		(fill
+			(color 0 0 0 0)
+		)
+		(property "Sheetname" "CHARGE"
+			(at 174.625 108.5084 0)
+			(show_name no)
+			(do_not_autoplace no)
+			(effects
+				(font
+					(size 1.27 1.27)
+				)
+				(justify left bottom)
+			)
+		)
+		(property "Sheetfile" "charge.kicad_sch"
+			(at 174.625 132.6646 0)
+			(show_name no)
+			(do_not_autoplace no)
+			(effects
+				(font
+					(size 1.27 1.27)
+				)
+				(justify left top)
+			)
+		)
+		(instances
+			(project "H616_devboard"
+				(path "/44f68964-8d75-4db0-b784-705712e148bc"
+					(page "7")
+				)
+			)
+		)
+	)
+	(sheet
+		(at 93.345 147.955)
+		(size 27.94 22.86)
+		(exclude_from_sim no)
+		(in_bom yes)
+		(on_board yes)
+		(dnp no)
+		(fields_autoplaced yes)
+		(stroke
+			(width 0.1524)
+			(type solid)
+		)
+		(fill
+			(color 0 0 0 0)
+		)
+		(property "Sheetname" "BOARD"
+			(at 93.345 147.2434 0)
+			(show_name no)
+			(do_not_autoplace no)
+			(effects
+				(font
+					(size 1.27 1.27)
+				)
+				(justify left bottom)
+			)
+		)
+		(property "Sheetfile" "board.kicad_sch"
+			(at 93.345 171.3996 0)
+			(show_name no)
+			(do_not_autoplace no)
+			(effects
+				(font
+					(size 1.27 1.27)
+				)
+				(justify left top)
+			)
+		)
+		(instances
+			(project "H616_devboard"
+				(path "/44f68964-8d75-4db0-b784-705712e148bc"
+					(page "8")
+				)
+			)
 		)
 	)
