File: Hardware/H616_DDR3/io1.kicad_sch (KiCad schematic)
At the start: 20 parts, among them J1 Micro_SD_Card_Det2, U1 H616

Commit message: v
Parts:
- removed R12, R13, R26: 10k, Resistor_SMD:R_0402_1005Metric_Pad0.72x0.64mm_HandSolder, symbol Device:R
- removed TP11, TP12, TP13: TestPoint, TestPoint:TestPoint_THTPad_D1.0mm_Drill0.5mm, symbol Connector:TestPoint
- added C82: 1u, Capacitor_SMD:C_0402_1005Metric_Pad0.74x0.62mm_HandSolder, symbol Device:C
- added C83, C85: 0.1u, Capacitor_SMD:C_0402_1005Metric_Pad0.74x0.62mm_HandSolder, symbol Device:C
- added C84: 2.2u, Capacitor_SMD:C_0402_1005Metric_Pad0.74x0.62mm_HandSolder, symbol Device:C
- added J2: HDMI_D_1.4, Connector_Video:HDMI_Micro-D_Molex_46765-1xxx, symbol Connector:HDMI_D_1.4
- added J5: Conn_01x40_Pin, HDR:DIP-30_100, symbol Connector:Conn_01x40_Pin
- added RN1, RN2, RN3: R_Pack04, Resistor_SMD:R_Array_Convex_4x0402, symbol Device:R_Pack04
- added U6: KLMBG2JETD-B041, Package_BGA:LFBGA-153_11.5x13mm_Layout14x14_P0.5mm, symbol JLCImport:KLMBG2JETD-B041
Connections:
- net +1V8: now also U1.F5 (VCC_PC), C82.1, C83.1, C85.1, RN1.5 (R4.2), RN1.6 (R3.2), RN1.7 (R2.2), RN1.8 (R1.2), RN2.5 (R4.2), RN2.6 (R3.2), RN2.7 (R2.2), RN2.8 (R1.2), RN3.7 (R2.2), RN3.8 (R1.2), U6.C2 (VDDI)
- net +3.3V: now also C84.1, RN3.5 (R4.2), RN3.6 (R3.2), U6.C6 (VDD), U6.E6 (VDDF), U6.F5 (VDDF), U6.J10 (VDDF), U6.K9 (VDDF), U6.M4 (VDD), U6.N4 (VDD), U6.P3 (VDD), U6.P5 (VDD); no longer U1.F5 (VCC_PC)
- net GND: now also C82.2, C83.2, C84.2, C85.2, U6.A6 (VSS), U6.C4 (VSS), U6.E7 (VSS), U6.G5 (VSS), U6.H10 (VSS), U6.J5 (VSS), U6.K8 (VSS), U6.N2 (VSS), U6.N5 (VSS), U6.P4 (VSS), U6.P6 (VSS)
- net SDC0_CMD: now also RN3.3 (R3.1)
- net SDC0_DET: now also RN3.4 (R4.1)
- net DATA-STROBE: now reaches U1.B1 (PC0)
- net DATA-STROBE: now also U6.H5 (DATA-STROBE)
- net EMMC_RSTN: now reaches U1.C2 (PC1)
- net EMMC_RSTN: now also RN1.1 (R1.1), U6.K5 (RSTN)
- net EMMC_CLK: now reaches U1.D3 (PC5)
- net EMMC_CLK: now also U6.M6 (CLK)
- net EMMC_CMD: now reaches U1.E2 (PC6)
- net EMMC_CMD: now also RN1.2 (R2.1), U6.M5 (CDM)
- net DAT0: now reaches U1.E3 (PC8)
- net DAT0: now also RN1.3 (R3.1), U6.A3 (DAT0)
- net DAT1: now reaches U1.F1 (PC9)
- net DAT1: now also RN1.4 (R4.1), U6.A4 (DAT1)
- net DAT2: now reaches U1.F2 (PC10)
- net DAT2: now also RN3.1 (R1.1), U6.A5 (DAT2)
- net DAT3: now reaches U1.F3 (PC11)
- net DAT3: now also RN3.2 (R2.1), U6.B2 (DAT3)
- net at U1.G2 (PC12): no longer R15.2
- net at R16.2: no longer U1.G3 (PC13)
- net DAT5: now reaches U1.H1 (PC14)
- net DAT5: now also RN2.2 (R2.1), U6.B4 (DAT5)
- net DAT6: now reaches U1.H2 (PC15)
- net DAT6: now also RN2.3 (R3.1), U6.B5 (DAT6)
- net DAT7: now reaches U1.H3 (PC16)
- net DAT7: now also RN2.4 (R4.1), U6.B6 (DAT7)
- new net DAT4: RN2.1 (R1.1), U1.G3 (PC13), U6.B3 (DAT4)
- no-connect marks 41 -> 31
Other:
- moved on the sheet: C51, D1, D2, J1, R10, R11, R14, R15, R16

Commit message: radio+hdr
Parts:
- removed J2: HDMI_D_1.4, Connector_Video:HDMI_Micro-D_Molex_46765-1xxx, symbol Connector:HDMI_D_1.4
- added U10, U11: D3V3XA4B10LP, Package_DFN_QFN:Diodes_UDFN-10_1x2.5mm_P0.5mm, symbol Power_Protection:D3V3XA4B10LP
- C51, C52, C53, C82, C83, C84, C85: footprint Capacitor_SMD:C_0402_1005Metric_Pad0.74x0.62mm_HandSolder -> Capacitor_SMD:C_0402_1005Metric
- R10, R11, R14, R15, R16, R17, R18: footprint Resistor_SMD:R_0402_1005Metric_Pad0.72x0.64mm_HandSolder -> Resistor_SMD:R_0402_1005Metric
Connections:
- net MDC is gone; now on net PI14: U1.L6 (PI14)
- net MDIO is gone; now on net PI15: U1.L4 (PI15)
- net RXCTL is gone; now on net PI5: U1.H4 (PI5)
- net RXD0 is gone; now on net PI3: U1.E4 (PI3)
- net RXD1 is gone; now on net PI2: U1.G6 (PI2)
- net TXD0 is gone; now on net RX_PI10: U1.L5 (PI10)
- net TXD1 is gone; now on net TX_PI9: U1.D5 (PI9)
- net +1V8: now also J5.3 (Pin_3)
- net +3.3V: now also J5.1 (Pin_1), J5.2 (Pin_2)
- net GND: now also J5.21 (Pin_21), J5.22 (Pin_22), J5.4 (Pin_4), J5.7 (Pin_7), U10.3 (VSS), U10.8 (VSS), U11.3 (VSS), U11.8 (VSS)
- net RXConvIn: now also J5.10 (Pin_10)
- net TXConvOut: now also J5.9 (Pin_9)
- net PH9: now reaches U1.A12 (PH9)
- net PH9: now also J5.11 (Pin_11)
- net at U1.A14 (PH4): no longer names the net of U1.A14 (PH4)
- net PH7: now reaches U1.B12 (PH7)
- net PH7: now also J5.13 (Pin_13)
- net PH10: now reaches U1.B13 (PH10)
- net PH5: now reaches U1.B14 (PH5)
- net PH2: now reaches U1.B15 (PH2)
- net PH8: now reaches U1.C13 (PH8)
- net PH8: now also J5.12 (Pin_12)
- net PH6: now reaches U1.C14 (PH6)
- net PH6: now also J5.14 (Pin_14)
- net PH3: now reaches U1.C15 (PH3)
- net PI6: now reaches U1.H5 (PI6)
- net PI6: now also J5.30 (Pin_30)
- net PI14: now reaches J5.15 (Pin_15)
- net PI15: now reaches J5.16 (Pin_16)
- net PI3: now reaches J5.17 (Pin_17)
- net PI2: now reaches J5.18 (Pin_18)
- net TX_PI9: now reaches J5.19 (Pin_19)
- net RX_PI10: now reaches J5.20 (Pin_20)
- net D-_1: now reaches J5.23 (Pin_23)
- net D-_1: now also U10.2
- net D+_1: now reaches J5.24 (Pin_24)
- net D+_1: now also U10.1
- net D-_2: now reaches J5.25 (Pin_25)
- net D-_2: now also U10.5
- net D+_2: now reaches J5.26 (Pin_26)
- net D+_2: now also U10.4
- net D-_3: now reaches J5.27 (Pin_27)
- net D-_3: now also U11.2
- net D+_3: now reaches J5.28 (Pin_28)
- net D+_3: now also U11.1
- net PI5: now reaches J5.29 (Pin_29)
- net +5VP_0: now reaches J5.5 (Pin_5)
- net +5VP_0: now also J5.6 (Pin_6), J5.8 (Pin_8)
- net CLK125: no longer names the net of U1.E5 (PI13)
- net RXC: no longer names the net of U1.G5 (PI4)
- net RXD2 renamed PI1
- net RXD3 renamed PI0
- net TXC: no longer names the net of U1.K4 (PI11)
- net TXCTL: no longer names the net of U1.K5 (PI12)
- net TXD2: no longer names the net of U1.E6 (PI8)
- net TXD3: no longer names the net of U1.G4 (PI7)
- new net D+: U11.4
- new net D-: U11.5
- no-connect marks 31 -> 21

Commit message: pcb
Parts:
- added U7: AP6256, bodya:AP6255, symbol JLCImport:AP6256
Connections:
- net +1V8: now also U7.22 (VDDIO)
- net +3.3V: now also U7.9 (VBAT)
- net PG6: now reaches U1.A4 (PG6)
- net PG6: now also U7.43 (UART_RXD)
- net PG0: now reaches U1.A6 (PG0)
- net PG0: now also U7.17 (SDIO_DATA_CLK)
- net PG15: now reaches U1.A8 (PG15)
- net PG15: now also U7.6 (BT_WAKE)
- net PG11: now reaches U1.B10 (PG11)
- net PG11: now also U7.12 (WL_REG_ON)
- net PG9: now reaches U1.B3 (PG9)
- net PG9: now also U7.41 (UAR_RTS_N)
- net PG7: now reaches U1.B4 (PG7)
- net PG7: now also U7.42 (UART_TXD)
- net PG3: now reaches U1.B5 (PG3)
- net PG3: now also U7.19 (SDIO_DATA_1)
- net PG5: now reaches U1.B7 (PG5)
- net PG5: now also U7.15 (SDIO_DATA_3)
- net PG14: now reaches U1.B9 (PG14)
- net PG14: now also U7.7 (BT_HOST_WAKE)
- net PG13: now reaches U1.C10 (PG13)
- net PG13: now also U7.13 (WL_HOST_WAKE)
- net PG8: now reaches U1.C4 (PG8)
- net PG8: now also U7.44 (UART_CTS_N)
- net PG4: now reaches U1.C5 (PG4)
- net PG4: now also U7.14 (SDIO_DATA_2)
- net PG2: now reaches U1.C6 (PG2)
- net PG2: now also U7.18 (SDIO_DATA_0)
- net PG1: now reaches U1.C7 (PG1)
- net PG1: now also U7.16 (SDIO_DATA_CMD)
- net PG10: now reaches U1.C8 (PG10)
- net PG12: now reaches U1.C9 (PG12)
- net PG12: now also U7.34 (BT_REG_ON)
- no-connect marks 21 -> 5
Other:
- moved on the sheet: J5, U10, U11

Commit message: Fix critical hardware bugs: eMMC HS400, AXP305 power rails, SW6206 Kelvin sense, Type-C CC and hierarchy
Connections:
- net +1V8: now also U6.C6 (VDD), U6.M4 (VDD), U6.N4 (VDD), U6.P3 (VDD), U6.P5 (VDD); no longer C82.1, U6.C2 (VDDI)
- net +3.3V: no longer U6.C6 (VDD), U6.M4 (VDD), U6.N4 (VDD), U6.P3 (VDD), U6.P5 (VDD)
- new net VDDI: C82.1, U6.C2 (VDDI)
Changed lines of the file:
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@@
 	)
 	(symbol
-		(lib_id "power:+3.3V")
+		(lib_id "power:+1V8")
 		(at 102.87 100.33 270)
 		(unit 1)
@@
 			)
 		)
-		(property "Value" "+3.3V"
+		(property "Value" "+1V8"
 			(at 107.188 97.536 0)
 			(show_name no)
@@
 	)
 	(symbol
-		(lib_id "power:+3.3V")
+		(lib_id "power:+1V8")
 		(at 102.87 146.05 270)
 		(unit 1)
@@
 			)
 		)
-		(property "Value" "+3.3V"
+		(property "Value" "+1V8"
 			(at 107.188 143.256 0)
 			(show_name no)
@@
 		)
 	)
-	(symbol
-		(lib_id "power:+1V8")
-		(at 102.87 95.25 270)
-		(unit 1)
-		(body_style 1)
-		(exclude_from_sim no)
-		(in_bom yes)
-		(on_board yes)
-		(in_pos_files yes)
-		(dnp no)
-		(property "Reference" "#PWR0120"
-			(at 99.06 95.25 0)
-			(hide yes)
-			(show_name no)
-			(do_not_autoplace no)
-			(effects
-				(font
-					(size 1.27 1.27)
-				)
-			)
-		)
-		(property "Value" "+1V8"
-			(at 106.68 92.71 0)
-			(show_name no)
-			(do_not_autoplace no)
-			(effects
-				(font
-					(size 1.27 1.27)
-				)
-				(justify left)
-			)
-		)
-		(property "Footprint" ""
-			(at 102.87 95.25 0)
-			(hide yes)
-			(show_name no)
-			(do_not_autoplace no)
-			(effects
-				(font
-					(size 1.27 1.27)
-				)
-			)
-		)
-		(property "Datasheet" ""
-			(at 102.87 95.25 0)
-			(hide yes)
-			(show_name no)
-			(do_not_autoplace no)
-			(effects
-				(font
-					(size 1.27 1.27)
-				)
-			)
-		)
-		(property "Description" ""
-			(at 102.87 95.25 0)
-			(hide yes)
-			(show_name no)
-			(do_not_autoplace no)
-			(effects
-				(font
-					(size 1.27 1.27)
-				)
-			)
-		)
-		(pin "1"
-		)
-		(instances
-			(project "H616_devboard"
-				(path "/44f68964-8d75-4db0-b784-705712e148bc/2e182087-17c9-4f42-b165-52dadf9ce5a4"
-					(reference "#PWR0120")
-					(unit 1)
-				)
+	(label "VDDI"
+		(at 102.87 95.25 0)
+		(fields_autoplaced yes)
+		(effects
+			(font
+				(size 1.27 1.27)
 			)
+			(justify left bottom)
 		)
 	)
@@
 	)
 	(symbol
-		(lib_id "power:+3.3V")
+		(lib_id "power:+1V8")
 		(at 102.87 140.97 270)
 		(unit 1)
@@
 			)
 		)
-		(property "Value" "+3.3V"
+		(property "Value" "+1V8"
 			(at 107.188 138.176 0)
 			(show_name no)
@@
 	)
 	(symbol
-		(lib_id "power:+3.3V")
+		(lib_id "power:+1V8")
 		(at 102.87 130.81 270)
 		(unit 1)
@@
 			)
 		)
-		(property "Value" "+3.3V"
+		(property "Value" "+1V8"
 			(at 107.188 128.016 0)
 			(show_name no)
@@
 		)
 	)
-	(symbol
-		(lib_id "power:+1V8")
-		(at 55.88 140.97 0)
-		(unit 1)
-		(body_style 1)
-		(exclude_from_sim no)
-		(in_bom yes)
-		(on_board yes)
-		(in_pos_files yes)
-		(dnp no)
-		(property "Reference" "#PWR0142"
-			(at 55.88 144.78 0)
-			(hide yes)
-			(show_name no)
-			(do_not_autoplace no)
-			(effects
-				(font
-					(size 1.27 1.27)
-				)
-			)
-		)
-		(property "Value" "+1V8"
-			(at 53.34 137.16 0)
-			(show_name no)
-			(do_not_autoplace no)
-			(effects
-				(font
-					(size 1.27 1.27)
-				)
-				(justify left)
-			)
-		)
-		(property "Footprint" ""
-			(at 55.88 140.97 0)
-			(hide yes)
-			(show_name no)
-			(do_not_autoplace no)
-			(effects
-				(font
-					(size 1.27 1.27)
-				)
-			)
-		)
-		(property "Datasheet" ""
-			(at 55.88 140.97 0)
-			(hide yes)
-			(show_name no)
-			(do_not_autoplace no)
-			(effects
-				(font
-					(size 1.27 1.27)
-				)
-			)
-		)
-		(property "Description" ""
-			(at 55.88 140.97 0)
-			(hide yes)
-			(show_name no)
-			(do_not_autoplace no)
-			(effects
-				(font
-					(size 1.27 1.27)
-				)
-			)
-		)
-		(pin "1"
-		)
-		(instances
-			(project "H616_devboard"
-				(path "/44f68964-8d75-4db0-b784-705712e148bc/2e182087-17c9-4f42-b165-52dadf9ce5a4"
-					(reference "#PWR0142")
-					(unit 1)
-				)
+	(label "VDDI"
+		(at 55.88 140.97 90)
+		(fields_autoplaced yes)
+		(effects
+			(font
+				(size 1.27 1.27)
 			)
+			(justify left bottom)
 		)
 	)
@@
 	)
 	(symbol
-		(lib_id "power:+3.3V")
+		(lib_id "power:+1V8")
 		(at 102.87 151.13 270)
 		(unit 1)
@@
 			)
 		)
-		(property "Value" "+3.3V"
+		(property "Value" "+1V8"
 			(at 107.188 148.336 0)
 			(show_name no)
