File: Hardware/H616_DDR3/power.kicad_sch (KiCad schematic)
At the start: 55 parts, among them U1 H616, U3 AXP305

Commit message: trace
Parts:
- U3: footprint Package_DFN_QFN:QFN-56-1EP_7x7mm_P0.4mm_EP4x4mm -> Package_DFN_QFN:QFN-56-1EP_7x7mm_P0.4mm_EP4x4mm_ThermalVias
Changed lines of the file:
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@@
 			)
 		)
-		(property "Footprint" "Package_DFN_QFN:QFN-56-1EP_7x7mm_P0.4mm_EP4x4mm"
+		(property "Footprint" "Package_DFN_QFN:QFN-56-1EP_7x7mm_P0.4mm_EP4x4mm_ThermalVias"
 			(at 80.01 40.64 0)
-			(hide yes)
 			(show_name no)
 			(do_not_autoplace no)
