File: Hardware/H616_DDR3/usb_uart.kicad_sch (KiCad schematic)
At the start: 5 parts, among them J3 USB_C_Receptacle_USB2.0

Commit message: radio+hdr
Parts:
- C65: footprint Capacitor_SMD:C_0402_1005Metric_Pad0.74x0.62mm_HandSolder -> Capacitor_SMD:C_0402_1005Metric
- R23, R24: footprint Resistor_SMD:R_0402_1005Metric_Pad0.72x0.64mm_HandSolder -> Resistor_SMD:R_0402_1005Metric
Changed lines of the file:
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@@
 			)
 		)
-		(property "Footprint" "Resistor_SMD:R_0402_1005Metric_Pad0.72x0.64mm_HandSolder"
+		(property "Footprint" "Resistor_SMD:R_0402_1005Metric"
 			(at 159.385 115.57 0)
 			(hide yes)
@@
 			)
 		)
-		(property "Footprint" "Resistor_SMD:R_0402_1005Metric_Pad0.72x0.64mm_HandSolder"
+		(property "Footprint" "Resistor_SMD:R_0402_1005Metric"
 			(at 159.385 118.11 0)
 			(hide yes)
@@
 			)
 		)
-		(property "Footprint" "Capacitor_SMD:C_0402_1005Metric_Pad0.74x0.62mm_HandSolder"
+		(property "Footprint" "Capacitor_SMD:C_0402_1005Metric"
 			(at 164.7698 110.49 0)
 			(hide yes)

Commit message: Fix critical hardware bugs: eMMC HS400, AXP305 power rails, SW6206 Kelvin sense, Type-C CC and hierarchy
Parts:
- R23, R24: value 22k -> 5.1k
Connections:
- net GND: now also R23.1, R24.1
- net at C65.2, J3.A4 (VBUS), J3.A9 (VBUS)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: no longer D4.1 (K), R23.1, R24.1
Changed lines of the file:
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@@
-	)
-	(junction
-		(at 156.845 110.49)
-		(diameter 0)
-		(color 0 0 0 0)
 	)
 	(junction
@@
 	(wire
 		(pts
-			(xy 165.735 110.49) (xy 156.845 110.49)
+			(xy 125.73 114.3) (xy 118.11 114.3)
 		)
 		(stroke
@@
 	(wire
 		(pts
-			(xy 125.73 114.3) (xy 118.11 114.3)
+			(xy 156.845 115.57) (xy 156.845 118.11)
 		)
 		(stroke
@@
 	(wire
 		(pts
-			(xy 156.845 115.57) (xy 156.845 118.11)
+			(xy 147.32 110.49) (xy 149.225 110.49)
 		)
 		(stroke
@@
 	(wire
 		(pts
-			(xy 147.32 110.49) (xy 149.225 110.49)
+			(xy 156.845 125.73) (xy 165.735 125.73)
 		)
 		(stroke
@@
 	(wire
 		(pts
-			(xy 156.845 125.73) (xy 165.735 125.73)
+			(xy 165.735 123.19) (xy 165.735 125.73)
 		)
 		(stroke
@@
 	(wire
 		(pts
-			(xy 165.735 123.19) (xy 165.735 125.73)
+			(xy 156.845 128.27) (xy 165.735 128.27)
 		)
 		(stroke
@@
 	(wire
 		(pts
-			(xy 156.845 128.27) (xy 165.735 128.27)
-		)
-		(stroke
-			(width 0)
-			(type default)
-		)
-	)
-	(wire
-		(pts
 			(xy 161.925 118.11) (xy 165.735 118.11)
-		)
-		(stroke
-			(width 0)
-			(type default)
-		)
-	)
-	(wire
-		(pts
-			(xy 156.845 110.49) (xy 156.845 115.57)
 		)
 		(stroke
@@
 			)
 		)
-		(property "Value" "22k"
+		(property "Value" "5.1k"
 			(at 164.465 113.665 90)
 			(show_name no)
@@
 			)
 		)
-		(property "Value" "22k"
+		(property "Value" "5.1k"
 			(at 164.465 120.015 90)
 			(show_name no)
@@
 		)
 	)
+	(symbol
+		(lib_id "power:GND")
+		(at 156.845 115.57 270)
+		(unit 1)
+		(body_style 1)
+		(exclude_from_sim no)
+		(in_bom yes)
+		(on_board yes)
+		(in_pos_files yes)
+		(dnp no)
+		(fields_autoplaced yes)
+		(property "Reference" "#PWR0197"
+			(at 153.035 115.57 0)
+			(hide yes)
+			(show_name no)
+			(do_not_autoplace no)
+			(effects
+				(font
+					(size 1.27 1.27)
+				)
+			)
+		)
+		(property "Value" "GND"
+			(at 156.845 119.38 90)
+			(show_name no)
+			(do_not_autoplace no)
+			(effects
+				(font
+					(size 1.27 1.27)
+				)
+			)
+		)
+		(property "Footprint" ""
+			(at 156.845 115.57 0)
+			(hide yes)
+			(show_name no)
+			(do_not_autoplace no)
+			(effects
+				(font
+					(size 1.27 1.27)
+				)
+			)
+		)
+		(property "Datasheet" ""
+			(at 156.845 115.57 0)
+			(hide yes)
+			(show_name no)
+			(do_not_autoplace no)
+			(effects
+				(font
+					(size 1.27 1.27)
+				)
+			)
+		)
+		(property "Description" ""
+			(at 156.845 115.57 0)
+			(hide yes)
+			(show_name no)
+			(do_not_autoplace no)
+			(effects
+				(font
+					(size 1.27 1.27)
+				)
+			)
+		)
+		(pin "1"
+		)
+		(instances
+			(project "H616_devboard"
+				(path "/44f68964-8d75-4db0-b784-705712e148bc/95399e0d-575a-4500-9429-e4d55ac775b9"
+					(reference "#PWR0197")
+					(unit 1)
+				)
+			)
+		)
+	)
+	(sheet_instances
+		(path "/44f68964-8d75-4db0-b784-705712e148bc/95399e0d-575a-4500-9429-e4d55ac775b9"
+			(page "6")
+		)
+	)
