File: Hardware/H616_DDR3/H616_devboard.kicad_pcb (KiCad board)
At the start: 8 copper layers, 50 x 50 mm, 169 parts, among them J1 Micro_SD_Card_Det2, J2 HDMI_D_1.4, J3 USB_C_Receptacle_USB2.0, J4 USB_C_Receptacle_USB2.0, J5 Conn_01x40_Pin, Q1 AO3420_C358680, Q2 AO3401A, Q3 AO3401A, SW1 CK_KMS2xxG, U1 H616, U10 D3V3XA4B10LP, U11 D3V3XA4B10LP, U2 K4B8G1646D, U3 AXP305, U4 SW6206, U6 KLMBG2JETD-B041, U7 AP6256, U8 D3V3XA4B10LP, U9 D3V3XA4B10LP, Y1 24MHz

Commit message: ddr trace
Routing:
- net /DRAM/SCKE1: track 0.00 -> 1.40 mm
Changed lines of the file:
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@@
 		(net "/DRAM/SDQ25")
+	)
+	(segment
+		(start 95.432813 57.755898)
+		(end 96.555898 57.755898)
+		(width 0.0922)
+		(layer "F.Cu")
+		(net "/DRAM/SCKE1")
+	)
+	(segment
+		(start 96.555898 57.755898)
+		(end 96.75 57.95)
+		(width 0.0922)
+		(layer "F.Cu")
+		(net "/DRAM/SCKE1")
 	)
 	(via

Commit message: ddr trace
Routing:
- net /DRAM/SCKE1: track 1.40 -> 2.59 mm
Changed lines of the file:
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@@
+	)
+	(segment
+		(start 96.75 57.95)
+		(end 97.8 57.95)
+		(width 0.0922)
+		(layer "F.Cu")
+		(net "/DRAM/SCKE1")
 	)
 	(segment
@@
 		(width 0.0922)
 		(layer "F.Cu")
+		(net "/DRAM/SCKE1")
+	)
+	(segment
+		(start 97.8 57.95)
+		(end 97.9 57.85)
+		(width 0.0922)
+		(layer "F.Cu")

Commit message: ddr trace
Routing:
- net /DRAM/SCKE1: track 2.59 -> 4.88 mm
Changed lines of the file:
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@@
+	)
+	(segment
+		(start 97.875 57.875)
+		(end 99.425 57.875)
+		(width 0.0922)
+		(layer "F.Cu")
+		(net "/DRAM/SCKE1")
 	)
 	(segment
@@
 	(segment
 		(start 97.8 57.95)
+		(end 97.875 57.875)
+		(width 0.0922)
+		(layer "F.Cu")
+		(net "/DRAM/SCKE1")
+	)
+	(segment
+		(start 97.875 57.875)
 		(end 97.9 57.85)
 		(width 0.0922)
 		(layer "F.Cu")
+		(net "/DRAM/SCKE1")
+	)
+	(segment
+		(start 99.425 57.875)
+		(end 99.95 58.4)
+		(width 0.0922)
+		(layer "F.Cu")

Commit message: ddr trace
Routing:
- net /DRAM/SCKE1: track 4.88 -> 7.26 mm
Changed lines of the file:
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@@
+	)
+	(segment
+		(start 101.6 60.05)
+		(end 101.65 60.05)
+		(width 0.0922)
+		(layer "F.Cu")
+		(net "/DRAM/SCKE1")
 	)
 	(segment
@@
 	(segment
 		(start 99.425 57.875)
-		(end 99.95 58.4)
+		(end 101.6 60.05)
 		(width 0.0922)
 		(layer "F.Cu")

Commit message: ddr trace
Routing:
- net /DRAM/SCKE1: track 7.26 -> 8.94 mm
Changed lines of the file:
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@@
 	)
 	(segment
-		(start 97.875 57.875)
-		(end 99.425 57.875)
+		(start 99.425 57.875)
+		(end 101.6 60.05)
 		(width 0.0922)
 		(layer "F.Cu")
@@
 		(start 96.555898 57.755898)
 		(end 96.75 57.95)
+		(width 0.0922)
+		(layer "F.Cu")
+		(net "/DRAM/SCKE1")
+	)
+	(segment
+		(start 97.875 57.875)
+		(end 99.425 57.875)
 		(width 0.0922)
 		(layer "F.Cu")
@@
 	(segment
 		(start 101.6 60.05)
-		(end 101.65 60.05)
+		(end 103.25 60.05)
 		(width 0.0922)
 		(layer "F.Cu")
@@
 	)
 	(segment
-		(start 99.425 57.875)
-		(end 101.6 60.05)
+		(start 103.25 60.05)
+		(end 103.3 60.1)
 		(width 0.0922)
 		(layer "F.Cu")

Commit message: ddr trace
Routing:
- net /DRAM/SCKE1: track 8.94 -> 0.00 mm
