File: Hardware/H616_DDR3/_restore_backup_2026-10-01T19-43-58-595/H616_devboard.kicad_pcb (KiCad board)
At the start: 8 copper layers, 50 x 50 mm, 163 parts, among them J1 Micro_SD_Card_Det2, J2 HDMI_D_1.4, J3 USB_C_Receptacle_USB2.0, J4 USB_C_Receptacle_USB2.0, J5 Conn_01x40_Pin, Q1 AO3420_C358680, SW1 CK_KMS2xxG, U1 H616, U10 D3V3XA4B10LP, U11 D3V3XA4B10LP, U2 K4B8G1646D, U3 AXP305, U4 SW6206, U6 KLMBG2JETD-B041, U7 AP6256, U8 D3V3XA4B10LP, U9 D3V3XA4B10LP, Y1 24MHz

Commit message: pcb
Parts:
- R15, R16, U7: moved to B.Cu
- moved TP7 54.2 mm to (136.2, 81.6)
- moved R15 49.2 mm to (125.6, 61.2), turned to 90 degrees
- moved D1 47.0 mm to (125.6, 61.2)
- moved D2 44.6 mm to (125.6, 64.8), turned to 90 degrees
- moved R16 42.9 mm to (125.6, 64.8)
- moved TP6 32.9 mm to (58.0, 65.5)
- moved TP8 27.6 mm to (128.8, 78.2)
- moved TP1 25.1 mm to (61.5, 63.0)
- moved TP5 23.1 mm to (60.9, 65.7)
- moved TP4 22.7 mm to (125.4, 49.9)
- moved TP2 14.2 mm to (132.4, 82.6)
- moved TP3 7.13 mm to (125.3, 84.1)
- moved J1 2.18 mm to (75.5, 58.5)
- moved U7 1.03 mm to (77.5, 57.9)
