File: Hardware/H616_DDR3/_restore_backup_2026-10-01T19-43-58-595/io1.kicad_sch (KiCad schematic)
At the start: 26 parts, among them J1 Micro_SD_Card_Det2, J5 Conn_01x40_Pin, U1 H616, U10 D3V3XA4B10LP, U11 D3V3XA4B10LP, U6 KLMBG2JETD-B041, U7 AP6256

Commit message: pcb
Parts:
- J1: footprint bodya:sd-short -> Connector_Card:microSD_HC_Hirose_DM3AT-SF-PEJM5
Changed lines of the file:
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@@
 		)
 	)
-	(label "VDDI"
-		(at 102.87 95.25 0)
-		(effects
-			(font
-				(size 1.27 1.27)
-			)
-			(justify left bottom)
-		)
-	)
 	(label "PI2"
 		(at 372.11 147.32 180)
@@
 		)
 	)
-	(label "VDDI"
-		(at 55.88 140.97 90)
-		(effects
-			(font
-				(size 1.27 1.27)
-			)
-			(justify left bottom)
-		)
-	)
 	(label "DAT0"
 		(at 106.68 72.39 0)
@@
 			)
 		)
-		(property "Footprint" "bodya:sd-short"
+		(property "Footprint" "Connector_Card:microSD_HC_Hirose_DM3AT-SF-PEJM5"
 			(at 273.685 52.07 0)
 			(hide yes)
@@
 		)
 	)
+	(label "VDDI"
+		(at 102.87 95.25 0)
+		(fields_autoplaced yes)
+		(effects
+			(font
+				(size 1.27 1.27)
+			)
+			(justify left bottom)
+		)
+	)
 	(symbol
 		(lib_id "Device:C")
@@
 		)
 	)
+	(label "VDDI"
+		(at 55.88 140.97 90)
+		(fields_autoplaced yes)
+		(effects
+			(font
+				(size 1.27 1.27)
+			)
+			(justify left bottom)
+		)
+	)
