File: Hardware/H616_DDR3/_restore_backup_2026-10-04T21-08-41-253/H616_devboard.kicad_pcb (KiCad board)
At the start: 8 copper layers, 50 x 50 mm, 161 parts, among them J1 Micro_SD_Card_Det2, J2 HDMI_D_1.4, J3 USB_C_Receptacle_USB2.0, J4 USB_C_Receptacle_USB2.0, J5 Conn_01x40_Pin, Q1 AO3420_C358680, Q2 AO3401A, Q3 AO3401A, SW1 CK_KMS2xxG, U1 H616, U10 D3V3XA4B10LP, U11 D3V3XA4B10LP, U2 K4B8G1646D, U3 AXP305, U4 SW6206, U6 KLMBG2JETD-B041, U7 AP6256, U8 D3V3XA4B10LP, U9 D3V3XA4B10LP, Y1 24MHz

Commit message: trace
Parts:
- C1, C10, C11, C12, C13, C14, C15, C16, C17, C18, C19, C2, C20, C21, C22, C23, C24, C25, C26, C27, C28, C29, C3, C30, C31, C32, C33, C34, C35, C36, C37, C38, C39, C4, C40, C41, C42, C43, C44, C45, C46, C47, C48, C49, C5, C50, C51, C52, C53, C54, C55, C56, C57, C58, C59, C6, C60, C61, C62, C63, C64, C65, C66, C67, C68, C69, C7, C70, C71, C72, C73, C74, C75, C76, C77, C78, C79, C8, C80, C81, C82, C83, C84, C85, C86, C87, C88, C9: footprint bodya:C_0402_1005Metric -> Capacitor_SMD:C_0402_1005Metric
- L1, L2, L3, L4, L5, L6: footprint bodya:L_Changjiang_FNR252010S -> Inductor_SMD:L_Changjiang_FNR252010S
- R1, R10, R11, R14, R15, R16, R17, R18, R19, R2, R20, R21, R22, R23, R24, R25, R26, R27, R28, R29, R3, R30, R31, R32, R33, R34, R35, R36, R4, R5, R6, R7, R8, R9: footprint bodya:R_0402_1005Metric -> Resistor_SMD:R_0402_1005Metric
