File: Hardware/H616_DDR3/_restore_backup_2026-10-04T21-08-41-253/io1.kicad_sch (KiCad schematic)
At the start: 30 parts, among them J1 Micro_SD_Card_Det2, J5 Conn_01x40_Pin, Q2 AO3401A, Q3 AO3401A, U1 H616, U10 D3V3XA4B10LP, U11 D3V3XA4B10LP, U6 KLMBG2JETD-B041, U7 AP6256

Commit message: trace
Parts:
- removed Q2, Q3: AO3401A, Package_TO_SOT_SMD:SOT-23, symbol Transistor_FET:AO3401A
- removed R35, R36: 10k, Resistor_SMD:R_0402_1005Metric, symbol Device:R
Connections:
- net GND: now also D1.1 (K), D2.1 (K); no longer R15.2, R16.2
- net at D1.2 (A): now also R15.1
- net at D2.2 (A): now also R16.1
Other:
- moved on the sheet: D1, D2, R15, R16
